Commit message: Added motor control using Gazebo

File: src/petpal_description/urdf/core.urdf.xacro (robot description, xacro)
@@ -5,36 +5,22 @@
     <parent link="base_link" />
     <child link="chassis" />
-    <origin xyz="0.0 0.0 0.0" />
+    <origin xyz="0 0 0" rpy="0 0 0"/>
   </joint>
   <link name="chassis">
     <visual>
-      <origin
-        xyz="0 0 0"
-        rpy="0 0 0" />
+      <origin xyz="0 0 0" rpy="0 0 0" />
       <geometry>
-        <mesh
-          filename="package://$(find petpal_description)/urdf/meshes/visual/base_link.STL" />
+        <mesh filename="file://$(find petpal_description)/meshes/visual/base_link.STL" />
       </geometry>
-      <material
-        name="">
-        <color
-          rgba="0.752941176470588 0.752941176470588 0.752941176470588 1" />
-      </material>
     </visual>
     <collision>
-      <origin
-        xyz="0 0 0"
-        rpy="0 0 0" />
+      <origin xyz="0 0 0" rpy="0 0 0" />
       <geometry>
-        <mesh
-          filename="package://$(find petpal_description)/urdf/meshes/collision/base_link.STL" />
+        <mesh filename="file://$(find petpal_description)/meshes/collision/base_link.STL" />
       </geometry>
     </collision>
     <inertial>
-      <origin
-        xyz="0.113980972815983 -0.00184514624243108 -0.00154363234446762"
-        rpy="0 0 0" />
-      <mass
-        value="0.709809139841652" />
+      <origin xyz="0.113980972815983 -0.00184514624243108 -0.00154363234446762" rpy="0 0 0" />
+      <mass value="0.709809139841652" />
       <inertia
         ixx="0.00035253122649593"
@@ -46,12 +32,20 @@
     </inertial>
   </link>
-  <link
-    name="fl_wheel">
+  <link name="fl_wheel">
+    <visual>
+      <origin xyz="0 0 0" rpy="0 0 0" />
+      <geometry>
+        <mesh filename="file://$(find petpal_description)/meshes/visual/fl_wheel.STL" />
+      </geometry>
+    </visual>
+    <collision>
+      <origin xyz="0 0 0" rpy="0 0 0" />
+      <geometry>
+        <mesh filename="file://$(find petpal_description)/meshes/collision/fl_wheel.STL" />
+      </geometry>
+    </collision>
     <inertial>
-      <origin
-        xyz="-0.0056365 2.1791E-05 -0.00055398"
-        rpy="0 0 0" />
-      <mass
-        value="0.063936" />
+      <origin xyz="-0.0056365 2.1791E-05 -0.00055398" rpy="0 0 0" />
+      <mass value="0.063936" />
       <inertia
         ixx="9.1342E-05"
@@ -62,27 +56,4 @@
         izz="6.5302E-05" />
     </inertial>
-    <visual>
-      <origin
-        xyz="0 0 0"
-        rpy="0 0 0" />
-      <geometry>
-        <mesh
-          filename="package://$(find petpal_description)/urdf/meshes/visual/fl_wheel.STL" />
-      </geometry>
-      <material
-        name="">
-        <color
-          rgba="0.75294 0.75294 0.75294 1" />
-      </material>
-    </visual>
-    <collision>
-      <origin
-        xyz="0 0 0"
-        rpy="0 0 0" />
-      <geometry>
-        <mesh
-          filename="package://$(find petpal_description)/urdf/meshes/collision/fl_wheel.STL" />
-      </geometry>
-    </collision>
   </link>
   <joint name="fl_wheel_joint" type="continuous">
@@ -90,14 +61,22 @@
     <parent link="chassis" />
     <child link="fl_wheel" />
-    <axis xyz="-0.9952 0.003845 -0.097807" />
+    <axis xyz="0.9952 -0.003845 0.097807" />
   </joint>
-  <link
-    name="fr_wheel">
+  <link name="fr_wheel">
+    <visual>
+      <origin xyz="0 0 0" rpy="0 0 0" />
+      <geometry>
+        <mesh filename="file://$(find petpal_description)/meshes/visual/fr_wheel.STL" />
+      </geometry>
+    </visual>
+    <collision>
+      <origin xyz="0 0 0" rpy="0 0 0" />
+      <geometry>
+        <mesh filename="file://$(find petpal_description)/meshes/collision/fr_wheel.STL" />
+      </geometry>
+    </collision>
     <inertial>
-      <origin
-        xyz="-0.0056365 -2.1749E-05 -0.00055395"
-        rpy="0 0 0" />
-      <mass
-        value="0.063936" />
+      <origin xyz="-0.0056365 -2.1749E-05 -0.00055395" rpy="0 0 0" />
+      <mass value="0.063936" />
       <inertia
         ixx="9.1342E-05"
@@ -108,49 +87,27 @@
         izz="6.5302E-05" />
     </inertial>
+  </link>
+  <joint name="fr_wheel_joint" type="continuous">
+    <origin xyz="0.29551 -0.12352 -0.019409" rpy="0 0 -1.5708" />
+    <parent link="base_link" />
+    <child link="fr_wheel" />
+    <axis xyz="-0.9952 -0.003845 -0.097807" />
+  </joint>
+  <link name="bl_wheel">
     <visual>
-      <origin
-        xyz="0 0 0"
-        rpy="0 0 0" />
+      <origin xyz="0 0 0" rpy="0 0 0" />
       <geometry>
-        <mesh
-          filename="package://$(find petpal_description)/urdf/meshes/visual/fr_wheel.STL" />
+        <mesh filename="file://$(find petpal_description)/meshes/visual/bl_wheel.STL" />
       </geometry>
-      <material
-        name="">
-        <color
-          rgba="0.75294 0.75294 0.75294 1" />
-      </material>
     </visual>
     <collision>
-      <origin
-        xyz="0 0 0"
-        rpy="0 0 0" />
+      <origin xyz="0 0 0" rpy="0 0 0" />
       <geometry>
-        <mesh
-          filename="package://$(find petpal_description)/urdf/meshes/collision/fr_wheel.STL" />
+        <mesh filename="file://$(find petpal_description)/meshes/collision/bl_wheel.STL" />
       </geometry>
     </collision>
-  </link>
-  <joint
-    name="fr_wheel_joint"
-    type="continuous">
-    <origin
-      xyz="0.29551 -0.12352 -0.019409"
-      rpy="0 0 -1.5708" />
-    <parent
-      link="base_link" />
-    <child
-      link="fr_wheel" />
-    <axis
-      xyz="-0.9952 -0.003845 -0.097807" />
-  </joint>
-  <link
-    name="bl_wheel">
     <inertial>
-      <origin
-        xyz="-0.0056999 -1.7387E-09 -0.00021923"
-        rpy="0 0 0" />
-      <mass
-        value="0.067933" />
+      <origin xyz="-0.0056999 -1.7387E-09 -0.00021923" rpy="0 0 0" />
+      <mass value="0.067933" />
       <inertia
         ixx="9.4408E-05"
@@ -161,49 +118,27 @@
         izz="6.4958E-05" />
     </inertial>
+  </link>
+  <joint name="bl_wheel_joint" type="fixed">
+    <origin xyz="0 0.13803 -0.021899" rpy="0 0 1.5708" />
+    <parent link="base_link" />
+    <child link="bl_wheel" />
+    <axis xyz="0.99926 0 0.038434" />
+  </joint>
+  <link name="br_wheel">
     <visual>
-      <origin
-        xyz="0 0 0"
-        rpy="0 0 0" />
+      <origin xyz="0 0 0" rpy="0 0 0" />
       <geometry>
-        <mesh
-          filename="package://$(find petpal_description)/urdf/meshes/visual/bl_wheel.STL" />
+        <mesh filename="file://$(find petpal_description)/meshes/visual/br_wheel.STL" />
       </geometry>
-      <material
-        name="">
-        <color
-          rgba="0.75294 0.75294 0.75294 1" />
-      </material>
     </visual>
     <collision>
-      <origin
-        xyz="0 0 0"
-        rpy="0 0 0" />
+      <origin xyz="0 0 0" rpy="0 0 0" />
       <geometry>
-        <mesh
-          filename="package://$(find petpal_description)/urdf/meshes/collision/bl_wheel.STL" />
+        <mesh filename="file://$(find petpal_description)/meshes/collision/br_wheel.STL" />
       </geometry>
     </collision>
-  </link>
-  <joint
-    name="bl_wheel_joint"
-    type="continuous">
-    <origin
-      xyz="0 0.13803 -0.021899"
-      rpy="0 0 1.5708" />
-    <parent
-      link="base_link" />
-    <child
-      link="bl_wheel" />
-    <axis
-      xyz="-0.99926 0 -0.038434" />
-  </joint>
-  <link
-    name="br_wheel">
     <inertial>
-      <origin
-        xyz="-0.0056999 -3.4019E-10 -0.00021923"
-        rpy="0 0 0" />
-      <mass
-        value="0.067933" />
+      <origin xyz="-0.0056999 -3.4019E-10 -0.00021923" rpy="0 0 0" />
+      <mass value="0.067933" />
       <inertia
         ixx="9.4408E-05"
@@ -214,40 +149,25 @@
         izz="6.4958E-05" />
     </inertial>
-    <visual>
-      <origin
-        xyz="0 0 0"
-        rpy="0 0 0" />
-      <geometry>
-        <mesh
-          filename="package://$(find petpal_description)/urdf/meshes/visual/br_wheel.STL" />
-      </geometry>
-      <material
-        name="">
-        <color
-          rgba="0.75294 0.75294 0.75294 1" />
-      </material>
-    </visual>
-    <collision>
-      <origin
-        xyz="0 0 0"
-        rpy="0 0 0" />
-      <geometry>
-        <mesh
-          filename="package://$(find petpal_description)/urdf/meshes/collision/br_wheel.STL" />
-      </geometry>
-    </collision>
   </link>
-  <joint
-    name="br_wheel_joint"
-    type="continuous">
-    <origin
-      xyz="0 -0.13803 -0.021899"
-      rpy="0 0 -1.5708" />
-    <parent
-      link="base_link" />
-    <child
-      link="br_wheel" />
-    <axis
-      xyz="-0.99926 0 -0.038434" />
+  <joint name="br_wheel_joint" type="fixed">
+    <origin xyz="0 -0.13803 -0.021899" rpy="0 0 -1.5708" />
+    <parent link="base_link" />
+    <child link="br_wheel" />
+    <axis xyz="-0.99926 0 -0.038434" />
   </joint>
+  <gazebo reference="chassis">
+    <material>Gazebo/White</material>
+  </gazebo>
+  <gazebo reference="fl_wheel">
+    <material>Gazebo/Grey</material>
+  </gazebo>
+  <gazebo reference="fr_wheel">
+    <material>Gazebo/Grey</material>
+  </gazebo>
+  <gazebo reference="bl_wheel">
+    <material>Gazebo/Grey</material>
+  </gazebo>
+  <gazebo reference="br_wheel">
+    <material>Gazebo/Grey</material>
+  </gazebo>
 </robot>

File: src/petpal_description/urdf/petpal.urdf.xacro (robot description, xacro)
@@ -2,3 +2,4 @@
 <robot name="petpal" xmlns:xacro="http://www.ros.org/wiki/xacro">
   <xacro:include filename="$(find petpal_description)/urdf/core.urdf.xacro" ns="petpal" />
+  <xacro:include filename="$(find petpal_description)/urdf/gazebo_control.urdf.xacro" />
 </robot>

File: src/petpal_description/urdf/wheel.urdf.xacro (robot description, xacro)
@@ -2,59 +2,4 @@
 <robot xmlns:xacro="http://www.ros.org/wiki/xacro">
 	<xacro:macro name="front_wheel" params="mirror">
-		<link name="fl_wheel">
-			<inertial>
-				<origin
-					xyz="-0.0056365 2.1791E-05 -0.00055398"
-					rpy="0 0 0" />
-				<mass
-					value="0.063936" />
-				<inertia
-					ixx="9.1342E-05"
-					ixy="-1.0157E-07"
-					ixz="2.5841E-06"
-					iyy="6.5049E-05"
-					iyz="-1.0144E-08"
-					izz="6.5302E-05" />
-			</inertial>
-			<visual>
-				<origin
-					xyz="0 0 0"
-					rpy="0 0 0" />
-				<geometry>
-					<mesh
-						filename="package://$(find petpal_sim)/urdf/meshes/visual/fl_wheel.STL" />
-				</geometry>
-				<material
-					name="">
-					<color
-						rgba="0.75294 0.75294 0.75294 1" />
-				</material>
-			</visual>
-			<collision>
-				<origin
-					xyz="0 0 0"
-					rpy="0 0 0" />
-				<geometry>
-					<mesh
-						filename="package://$(find petpal_sim)/urdf/meshes/collision/fl_wheel.STL" />
-				</geometry>
-			</collision>
-		</link>
-		<joint name="fl_wheel_joint" type="revolute">
-			<origin
-				xyz="0.29551 0.12352 -0.019409"
-				rpy="0 0 1.5708" />
-			<parent
-				link="base_link" />
-			<child
-				link="fl_wheel" />
-			<axis
-				xyz="-0.9952 0.003845 -0.097807" />
-			<limit
-				lower="0"
-				upper="0"
-				effort="0"
-				velocity="0" />
-		</joint>
 	</xacro:macro>
 </robot>
